File: hardware-atx-psu-12v-led/mainboard.kicad_pcb (KiCad board)
At the start: 2 copper layers, 98 x 103 mm, 100 parts, among them J1 ATX-24, J11 LED, J12 LED, J13 LED, J14 LED, J15 LED, J16 LED, J17 LED, J18 LED, J19 LED, J2 ATX, J20 LED, J21 LED, J22 LED, J23 LED, J24 LED, J25 LED, J26 LED, J27 LED, J28 LED, J29 LED, J3 PA11, J30 LED, J31 LED, J32 LED, J33 LED, J34 LED, J35 LED, J36 LED, J37 LED, J38 LED, J39 LED, J4 PA12, J40 LED, J41 LED, J42 ATX, J43 ATX, J44 ATX, J45 ATX, J5 LED, J6 USB_C_Receptacle_USB2.0, J7 PAGM, J8 PA15, SW1 Download, U1 CH32V305RBT6, U2 AMS1117, Y2 8MHz

Commit message: Add revB
Other:
- board text added: "-D+ x32"
- board text added: "x32-ws2812-usbhs-breakout hardware-atx-psu-12v-led rev B"
- board text removed: "cnhardware xmastree mainboard rev A"
Changed lines of the file:
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@@
 			(drillshape 0)
 			(scaleselection 1)
-			(outputdirectory "mainboard-revA/")
+			(outputdirectory "mainboard-revB/")
 		)
 	)
@@
 			(at 0 0.6)
 			(size 2.7 3.3)
-			(drill 1.4)
+			(drill 1.55)
 			(layers "*.Cu" "*.Mask")
 			(remove_unused_layers no)
@@
 			(at 4.2 0.6)
 			(size 2.7 3.3)
-			(drill 1.4)
+			(drill 1.55)
 			(layers "*.Cu" "*.Mask")
 			(remove_unused_layers no)
@@
 			(at 8.4 0.6)
 			(size 2.7 3.3)
-			(drill 1.4)
+			(drill 1.55)
 			(layers "*.Cu" "*.Mask")
 			(remove_unused_layers no)
@@
 			(at 12.6 0.6)
 			(size 2.7 3.3)
-			(drill 1.4)
+			(drill 1.55)
 			(layers "*.Cu" "*.Mask")
 			(remove_unused_layers no)
@@
 			(at 0 4.9)
 			(size 2.7 3.3)
-			(drill 1.4)
+			(drill 1.55)
 			(layers "*.Cu" "*.Mask")
 			(remove_unused_layers no)
@@
 			(at 4.2 4.9)
 			(size 2.7 3.3)
-			(drill 1.4)
+			(drill 1.55)
 			(layers "*.Cu" "*.Mask")
 			(remove_unused_layers no)
@@
 			(at 8.4 4.9)
 			(size 2.7 3.3)
-			(drill 1.4)
+			(drill 1.55)
 			(layers "*.Cu" "*.Mask")
 			(remove_unused_layers no)
@@
 			(at 12.6 4.9)
 			(size 2.7 3.3)
-			(drill 1.4)
+			(drill 1.55)
 			(layers "*.Cu" "*.Mask")
 			(remove_unused_layers no)
@@
 			(at 0 0.6 270)
 			(size 2.7 3.3)
-			(drill 1.4)
+			(drill 1.55)
 			(layers "*.Cu" "*.Mask")
 			(remove_unused_layers no)
@@
 			(at 4.2 0.6 270)
 			(size 2.7 3.3)
-			(drill 1.4)
+			(drill 1.55)
 			(layers "*.Cu" "*.Mask")
 			(remove_unused_layers no)
@@
 			(at 8.4 0.6 270)
 			(size 2.7 3.3)
-			(drill 1.4)
+			(drill 1.55)
 			(layers "*.Cu" "*.Mask")
 			(remove_unused_layers no)
@@
 			(at 12.6 0.6 270)
 			(size 2.7 3.3)
-			(drill 1.4)
+			(drill 1.55)
 			(layers "*.Cu" "*.Mask")
 			(remove_unused_layers no)
@@
 			(at 0 4.9 270)
 			(size 2.7 3.3)
-			(drill 1.4)
+			(drill 1.55)
 			(layers "*.Cu" "*.Mask")
 			(remove_unused_layers no)
@@
 			(at 4.2 4.9 270)
 			(size 2.7 3.3)
-			(drill 1.4)
+			(drill 1.55)
 			(layers "*.Cu" "*.Mask")
 			(remove_unused_layers no)
@@
 			(at 8.4 4.9 270)
 			(size 2.7 3.3)
-			(drill 1.4)
+			(drill 1.55)
 			(layers "*.Cu" "*.Mask")
 			(remove_unused_layers no)
@@
 			(at 12.6 4.9 270)
 			(size 2.7 3.3)
-			(drill 1.4)
+			(drill 1.55)
 			(layers "*.Cu" "*.Mask")
 			(remove_unused_layers no)
@@
 			(at 0 0.6 270)
 			(size 2.7 3.3)
-			(drill 1.4)
+			(drill 1.55)
 			(layers "*.Cu" "*.Mask")
 			(remove_unused_layers no)
@@
 			(at 4.2 0.6 270)
 			(size 2.7 3.3)
-			(drill 1.4)
+			(drill 1.55)
 			(layers "*.Cu" "*.Mask")
 			(remove_unused_layers no)
@@
 			(at 8.4 0.6 270)
 			(size 2.7 3.3)
-			(drill 1.4)
+			(drill 1.55)
 			(layers "*.Cu" "*.Mask")
 			(remove_unused_layers no)
@@
 			(at 12.6 0.6 270)
 			(size 2.7 3.3)
-			(drill 1.4)
+			(drill 1.55)
 			(layers "*.Cu" "*.Mask")
 			(remove_unused_layers no)
@@
 			(at 0 4.9 270)
 			(size 2.7 3.3)
-			(drill 1.4)
+			(drill 1.55)
 			(layers "*.Cu" "*.Mask")
 			(remove_unused_layers no)
@@
 			(at 4.2 4.9 270)
 			(size 2.7 3.3)
-			(drill 1.4)
+			(drill 1.55)
 			(layers "*.Cu" "*.Mask")
 			(remove_unused_layers no)
@@
 			(at 8.4 4.9 270)
 			(size 2.7 3.3)
-			(drill 1.4)
+			(drill 1.55)
 			(layers "*.Cu" "*.Mask")
 			(remove_unused_layers no)
@@
 			(at 12.6 4.9 270)
 			(size 2.7 3.3)
-			(drill 1.4)
+			(drill 1.55)
 			(layers "*.Cu" "*.Mask")
 			(remove_unused_layers no)
@@
 			(at 0 0.6 270)
 			(size 2.7 3.3)
-			(drill 1.4)
+			(drill 1.55)
 			(layers "*.Cu" "*.Mask")
 			(remove_unused_layers no)
@@
 			(at 4.2 0.6 270)
 			(size 2.7 3.3)
-			(drill 1.4)
+			(drill 1.55)
 			(layers "*.Cu" "*.Mask")
 			(remove_unused_layers no)
@@
 			(at 8.4 0.6 270)
 			(size 2.7 3.3)
-			(drill 1.4)
+			(drill 1.55)
 			(layers "*.Cu" "*.Mask")
 			(remove_unused_layers no)
@@
 			(at 12.6 0.6 270)
 			(size 2.7 3.3)
-			(drill 1.4)
+			(drill 1.55)
 			(layers "*.Cu" "*.Mask")
 			(remove_unused_layers no)
@@
 			(at 0 4.9 270)
 			(size 2.7 3.3)
-			(drill 1.4)
+			(drill 1.55)
 			(layers "*.Cu" "*.Mask")
 			(remove_unused_layers no)
@@
 			(at 4.2 4.9 270)
 			(size 2.7 3.3)
-			(drill 1.4)
+			(drill 1.55)
 			(layers "*.Cu" "*.Mask")
 			(remove_unused_layers no)
@@
 			(at 8.4 4.9 270)
 			(size 2.7 3.3)
-			(drill 1.4)
+			(drill 1.55)
 			(layers "*.Cu" "*.Mask")
 			(remove_unused_layers no)
@@
 			(at 12.6 4.9 270)
 			(size 2.7 3.3)
-			(drill 1.4)
+			(drill 1.55)
 			(layers "*.Cu" "*.Mask")
 			(remove_unused_layers no)
@@
 			(at 0 0.6 180)
 			(size 2.7 3.3)
-			(drill 1.4)
+			(drill 1.55)
 			(layers "*.Cu" "*.Mask")
 			(remove_unused_layers no)
@@
 			(at 4.2 0.6 180)
 			(size 2.7 3.3)
-			(drill 1.4)
+			(drill 1.55)
 			(layers "*.Cu" "*.Mask")
 			(remove_unused_layers no)
@@
 			(at 8.4 0.6 180)
 			(size 2.7 3.3)
-			(drill 1.4)
+			(drill 1.55)
 			(layers "*.Cu" "*.Mask")
 			(remove_unused_layers no)
@@
 			(at 12.6 0.6 180)
 			(size 2.7 3.3)
-			(drill 1.4)
+			(drill 1.55)
 			(layers "*.Cu" "*.Mask")
 			(remove_unused_layers no)
@@
 			(at 0 4.9 180)
 			(size 2.7 3.3)
-			(drill 1.4)
+			(drill 1.55)
 			(layers "*.Cu" "*.Mask")
 			(remove_unused_layers no)
@@
 			(at 4.2 4.9 180)
 			(size 2.7 3.3)
-			(drill 1.4)
+			(drill 1.55)
 			(layers "*.Cu" "*.Mask")
 			(remove_unused_layers no)
@@
 			(at 8.4 4.9 180)
 			(size 2.7 3.3)
-			(drill 1.4)
+			(drill 1.55)
 			(layers "*.Cu" "*.Mask")
 			(remove_unused_layers no)
@@
 			(at 12.6 4.9 180)
 			(size 2.7 3.3)
-			(drill 1.4)
+			(drill 1.55)
 			(layers "*.Cu" "*.Mask")
 			(remove_unused_layers no)
@@
 		)
 	)
-	(gr_text "cnhardware\nxmastree\nmainboard\nrev A"
-		(at 150.82 59.18 0)
+	(gr_text "x32-ws2812-usbhs-breakout\nhardware-atx-psu-12v-led\nrev B"
+		(at 150 59 90)
 		(layer "F.SilkS")
 		(effects
 			(font
-				(size 1.5 1.5)
+				(size 1.3 1.3)
 				(thickness 0.3)
 				(bold yes)
@@
 		)
 	)
+	(gr_text "-D+ x32"
+		(at 115.5 66 0)
+		(layer "F.SilkS")
+		(effects
+			(font
+				(size 2.2 2.2)
+				(thickness 0.4)
+				(bold yes)
+			)
+			(justify left bottom)
+		)
+	)
