File: hardware-atx-psu-12v-led/mainboard.kicad_sch (KiCad schematic)
At the start: 100 parts, among them J1 ATX-24, J11 LED, J12 LED, J13 LED, J14 LED, J15 LED, J16 LED, J17 LED, J18 LED, J19 LED, J2 ATX, J20 LED, J21 LED, J22 LED, J23 LED, J24 LED, J25 LED, J26 LED, J27 LED, J28 LED, J29 LED, J3 PA11, J30 LED, J31 LED, J32 LED, J33 LED, J34 LED, J35 LED, J36 LED, J37 LED, J38 LED, J39 LED, J4 PA12, J40 LED, J41 LED, J42 ATX, J43 ATX, J44 ATX, J45 ATX, J5 LED, J6 USB_C_Receptacle_USB2.0, J7 PAGM, J8 PA15, SW1 Download, U1 CH32V305RBT6, U2 AMS1117, Y2 8MHz

Commit message: Add revB
Parts:
- J3, J4, J8: now not fitted
Other:
- note added: "Rev A: 1. USB to PB 2. Use PA6/7 instead of PB6/7 3. Use correct connector for PCI-E Rev B: 1. Fix hole sizes for PCI-E"
- note removed: "Rev A: 1. USB to PB 2. Use PA6/7 3. Fixed"
Changed lines of the file:
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@@
 	(generator_version "9.0")
 	(paper "A4")
-	(text "Rev A:\n1. USB to PB\n2. Use PA6/7\n3. Fixed"
+	(text "Rev A:\n1. USB to PB\n2. Use PA6/7 instead of PB6/7\n3. Use correct connector for PCI-E\n\nRev B:\n1. Fix hole sizes for PCI-E"
 		(exclude_from_sim no)
-		(at 157.226 141.224 0)
+		(at 133.096 135.636 0)
 		(effects
 			(font
@@
 				(thickness 0.1588)
 			)
+			(justify left top)
 		)
 	)
@@
 		(in_bom no)
 		(on_board yes)
-		(dnp no)
+		(dnp yes)
 		(fields_autoplaced yes)
 		(property "Reference" "J3"
@@
 		(in_bom no)
 		(on_board yes)
-		(dnp no)
+		(dnp yes)
 		(fields_autoplaced yes)
 		(property "Reference" "J8"
@@
 		(in_bom no)
 		(on_board yes)
-		(dnp no)
+		(dnp yes)
 		(fields_autoplaced yes)
 		(property "Reference" "J4"
