File: hardware-atx-psu-12v-led/mainboard.kicad_sch (KiCad schematic)
At the start: 100 parts, among them J1 ATX-24, J11 LED, J12 LED, J13 LED, J14 LED, J15 LED, J16 LED, J17 LED, J18 LED, J19 LED, J2 ATX, J20 LED, J21 LED, J22 LED, J23 LED, J24 LED, J25 LED, J26 LED, J27 LED, J28 LED, J29 LED, J3 PA11, J30 LED, J31 LED, J32 LED, J33 LED, J34 LED, J35 LED, J36 LED, J37 LED, J38 LED, J39 LED, J4 PA12, J40 LED, J41 LED, J42 ATX, J43 ATX, J44 ATX, J45 ATX, J5 LED, J6 USB_C_Receptacle_USB2.0, J7 PAGM, J8 PA15, SW1 Download, U1 CH32V305RBT6, U2 AMS1117, Y2 8MHz

Commit message: bump design
Connections:
- net 12V1: now also J18.3 (Pin_3), J19.3 (Pin_3), J20.3 (Pin_3), J23.3 (Pin_3), J24.3 (Pin_3), J25.3 (Pin_3); no longer J11.3 (Pin_3), J12.3 (Pin_3), J13.3 (Pin_3), J14.3 (Pin_3), J15.3 (Pin_3), J5.3 (Pin_3)
- net 12V2: now also J11.3 (Pin_3), J12.3 (Pin_3), J13.3 (Pin_3), J14.3 (Pin_3), J15.3 (Pin_3); no longer J17.3 (Pin_3), J18.3 (Pin_3), J19.3 (Pin_3), J20.3 (Pin_3), J21.3 (Pin_3)
- net 12V3: now also J17.3 (Pin_3), J32.3 (Pin_3), J33.3 (Pin_3), J5.3 (Pin_3); no longer J22.3 (Pin_3), J23.3 (Pin_3), J24.3 (Pin_3), J25.3 (Pin_3)
- net 12V4: now also J34.3 (Pin_3), J41.3 (Pin_3); no longer J32.3 (Pin_3), J33.3 (Pin_3)
- net 12V5: now also J40.3 (Pin_3); no longer J34.3 (Pin_3)
- net 12V6: now also J21.3 (Pin_3), J22.3 (Pin_3); no longer J40.3 (Pin_3), J41.3 (Pin_3)
